Commit message: After setting the environment

File: helpers/turtlebot/turtlebot3_waffle.urdf.xacro (robot description, xacro)
@@ -215,30 +215,3 @@
   </joint>
   <link name="camera_depth_optical_frame"/>
-  <link name="stand">
-    <visual>
-     <origin xyz="-0.15 -0.15 0.007" rpy="0 0 0"/>
-     <geometry>
-       <mesh filename="package://turtlebot3_description/meshes/basket/basket.dae" scale="1 1 0.5"/>
-     </geometry>
-    </visual>
-   <collision>
-      <origin xyz="-0.15 -0.15 0.007" rpy="0 0 0"/>
-     <geometry>
-       <mesh filename="package://turtlebot3_description/meshes/basket/basket.dae" scale="1 1 0.5"/>
-     </geometry>
-      <surface>
-        <friction>
-         <ode>
-            <mu>1000</mu>
-            <mu2>1000</mu2>
-          </ode>
-        </friction>
-      </surface>
-    </collision>
-  </link>
-  <joint name="stand_joint" type="fixed">
-     <parent link="base_scan"/>
-     <child link="stand"/>
-     <origin xyz="0 0 0.010"/>
-  </joint>
 </robot>
